File: HackPad.kicad_pcb (KiCad board)
At the start: 2 copper layers, 78.1 x 95.7 mm, 54 parts, among them SW1 SW_Push, SW10 SW_Push, SW11 SW_Push, SW12 SW_Push, SW13 SW_Push, SW14 SW_Push, SW15 SW_Push, SW16 SW_Push, SW17 RotaryEncoder_Switch, SW2 SW_Push, SW3 SW_Push, SW4 SW_Push, SW5 SW_Push, SW6 SW_Push, SW7 SW_Push, SW8 SW_Push, SW9 SW_Push, U1 MOUDLE-SEEEDUINO-XIAO, U2 ER_OLEDM0.91_1x-I2C

Commit message: remove knob
Parts:
- removed D17: 1N4148, Diode_THT:D_DO-35_SOD27_P7.62mm_Horizontal
- removed SW17: RotaryEncoder_Switch, Library:RotaryEncoder_Alps_EC11E-Switch_Vertical_H20mm
- moved L13 4.33 mm to (77.7, 108.0)
- moved L1 4.32 mm to (77.5, 50.0)
- moved L2 4.32 mm to (96.8, 50.0)
- moved L3 4.32 mm to (116.1, 50.0)
- moved L4 4.32 mm to (135.4, 50.0)
- moved L10 4.32 mm to (96.8, 88.6)
- moved L11 4.32 mm to (116.1, 88.6)
- moved L12 4.32 mm to (135.4, 88.6)
- moved L14 4.32 mm to (96.8, 108.0)
- moved L15 4.32 mm to (116.1, 108.0)
- moved L16 4.32 mm to (135.4, 108.0)
- moved L5 4.32 mm to (77.5, 69.3)
- moved L6 4.32 mm to (96.8, 69.3)
- moved L7 4.32 mm to (116.1, 69.3)
- moved L8 4.32 mm to (135.4, 69.3)
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Connections:
- D1 pad 1: /P2 -> /W5
- D10 pad 1: /P2 -> /W7
- D11 pad 1: /P4 -> /W7
- D12 pad 1: /P5 -> /W7
- D13 pad 1: /P1 -> /W8
- D14 pad 1: /P2 -> /W8
- D15 pad 1: /P3 -> /W8
- D16 pad 1: /P5 -> /W8
- D2 pad 1: /P3 -> /W5
- D3 pad 1: /P4 -> /W5
- D4 pad 1: /P5 -> /W5
- D5 pad 1: /P1 -> /W6
- D6 pad 1: /P3 -> /W6
- D7 pad 1: /P4 -> /W6
- D8 pad 1: /P5 -> /W6
- D9 pad 1: /P1 -> /W7
- SW1 pad 1: /P1 -> /W1
- SW10 pad 1: /P3 -> /W2
- SW11 pad 1: /P3 -> /W3
- SW12 pad 1: /P3 -> /W4
- SW13 pad 1: /P4 -> /W1
- SW14 pad 1: /P4 -> /W2
- SW15 pad 1: /P4 -> /W3
- SW16 pad 1: /P4 -> /W4
- SW2 pad 1: /P1 -> /W2
- SW3 pad 1: /P1 -> /W3
- SW4 pad 1: /P1 -> /W4
- SW5 pad 1: /P2 -> /W1
- SW6 pad 1: /P2 -> /W2
- SW7 pad 1: /P2 -> /W3
- SW8 pad 1: /P2 -> /W4
- SW9 pad 1: /P3 -> /W1
- U1 pad 10: /P2 -> /W6
- U1 pad 11: /P1 -> /W5
- U1 pad 2: Net-(U1-PA4_A1_D1) -> /W1
- U1 pad 3: Net-(U1-PA10_A2_D2) -> /W2
- U1 pad 4: unconnected-(U1-PA11_A3_D3-Pad4) -> /W3
- U1 pad 7: /P5 -> /W4
- U1 pad 8: /P4 -> /W8
- U1 pad 9: /P3 -> /W7
Routing:
- net /P1: track 271.1 -> 0.00 mm, vias 14 -> 0
- net /P2: track 225.0 -> 0.00 mm, vias 7 -> 0
- net /P4: track 202.7 -> 0.00 mm
- net /P3: track 168.4 -> 0.00 mm, vias 4 -> 0
- net /W8: track 0.00 -> 136.8 mm, vias 0 -> 1
- net /W7: track 0.00 -> 133.7 mm, vias 0 -> 3
- net /W1: track 0.00 -> 122.6 mm
- net /W6: track 0.00 -> 115.4 mm, vias 0 -> 1
- net /W2: track 0.00 -> 101.1 mm
- net /P5: track 97.7 -> 0.00 mm
- net /W5: track 0.00 -> 90.3 mm
- net /W4: track 0.00 -> 72.3 mm
- net /W3: track 0.00 -> 68.5 mm
- net Net-(D17-A): track 14.5 -> 0.00 mm
- net Net-(L1-DIN): track 90.3 -> 79.2 mm, vias 0 -> 2
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