File: HackPad.kicad_sch (KiCad schematic)
At the start: 54 parts, among them SW1 SW_Push, SW10 SW_Push, SW11 SW_Push, SW12 SW_Push, SW13 SW_Push, SW14 SW_Push, SW15 SW_Push, SW16 SW_Push, SW17 RotaryEncoder_Switch, SW2 SW_Push, SW3 SW_Push, SW4 SW_Push, SW5 SW_Push, SW6 SW_Push, SW7 SW_Push, SW8 SW_Push, SW9 SW_Push, U1 MOUDLE-SEEEDUINO-XIAO, U2 ER_OLEDM0.91_1x-I2C

Commit message: remove knob
Parts:
- removed D17: 1N4148, Diode_THT:D_DO-35_SOD27_P7.62mm_Horizontal, symbol Diode:1N4148
- removed SW17: RotaryEncoder_Switch, Library:RotaryEncoder_Alps_EC11E-Switch_Vertical_H20mm, symbol Device:RotaryEncoder_Switch
Connections:
- net W1: now reaches U1.2 (PA4_A1_D1)
- net W1: now also SW1.1, SW13.1, SW5.1, SW9.1
- net W2: now reaches U1.3 (PA10_A2_D2)
- net W2: now also SW10.1, SW14.1, SW2.1, SW6.1
- net W3: now reaches U1.4 (PA11_A3_D3)
- net W3: now also SW11.1, SW15.1, SW3.1, SW7.1
- removed net P1: D13.1 (K), D5.1 (K), D9.1 (K), SW1.1, SW2.1, SW3.1, SW4.1, U1.11 (PA6_A10_D10_MOSI)
- removed net P2: D1.1 (K), D10.1 (K), D14.1 (K), SW5.1, SW6.1, SW7.1, SW8.1, U1.10 (PA5_A9_D9_MISO)
- removed net P3: D15.1 (K), D2.1 (K), D6.1 (K), SW10.1, SW11.1, SW12.1, SW9.1, U1.9 (PA7_A8_D8_SCK)
- removed net P4: D11.1 (K), D3.1 (K), D7.1 (K), SW13.1, SW14.1, SW15.1, SW16.1, U1.8 (PB09_A7_D7_RX)
- removed net P5: D12.1 (K), D16.1 (K), D4.1 (K), D8.1 (K), U1.7 (PB08_A6_D6_TX)
- new net W4: SW12.1, SW16.1, SW4.1, SW8.1, U1.7 (PB08_A6_D6_TX)
- new net W5: D1.1 (K), D2.1 (K), D3.1 (K), D4.1 (K), U1.11 (PA6_A10_D10_MOSI)
- new net W6: D5.1 (K), D6.1 (K), D7.1 (K), D8.1 (K), U1.10 (PA5_A9_D9_MISO)
- new net W7: D10.1 (K), D11.1 (K), D12.1 (K), D9.1 (K), U1.9 (PA7_A8_D8_SCK)
- new net W8: D13.1 (K), D14.1 (K), D15.1 (K), D16.1 (K), U1.8 (PB09_A7_D7_RX)
